File: hardware/ACS DB.sch (KiCad schematic (older format))
At the start: 41 parts, among them IC1 USR-ES1, J1 Power, J2 Reader 2, J3 Reader 1, J4 Relay 1, J5 Sensor 1, J6 Relay 2, J7 Sensor 2, J8 PB2, J9 PB1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

Commit message: update pcb layout
Parts:
- added H1, H2, H3, H4: MountingHole, MountingHole:MountingHole_3.2mm_M3, symbol Mechanical:MountingHole
- C1: footprint (none) -> Capacitor_SMD:CP_Elec_10x10
- C2: footprint (none) -> Capacitor_SMD:CP_Elec_6.3x7.7
- D1: value SS54 -> SS34; footprint (none) -> Diode_SMD:D_SMA_Handsoldering
- D10, D11, D12, D13, D14, D15, D16, D7, D8, D9: footprint (none) -> Diode_SMD:D_SMA_Handsoldering
- D2, D3, D4, D5, D6: footprint (none) -> LED_THT:LED_D5.0mm
- F1, F2: footprint (none) -> Resistor_SMD:R_1812_4532Metric_Pad1.30x3.40mm_HandSolder
- IC1: footprint USRES1 -> user-libraries:USRES1
- J1, J5, J7, J8, J9: footprint (none) -> Connector_Phoenix_MC_HighVoltage:PhoenixContact_MC_1,5_2-G-5.08_1x02_P5.08mm_Horizontal
- J2, J3: footprint (none) -> Connector_Phoenix_MC_HighVoltage:PhoenixContact_MC_1,5_5-G-5.08_1x05_P5.08mm_Horizontal
- J4, J6: footprint (none) -> Connector_Phoenix_MC_HighVoltage:PhoenixContact_MC_1,5_3-G-5.08_1x03_P5.08mm_Horizontal
- L1: footprint (none) -> Inductor_SMD:L_12x12mm_H6mm
- R1, R2, R3, R4, R5: footprint (none) -> Resistor_SMD:R_0805_2012Metric_Pad1.15x1.40mm_HandSolder
- U2: footprint (none) -> Package_TO_SOT_THT:TO-92_HandSolder
- U3: footprint (none) -> Package_SO:SOIC-18W_7.5x11.6mm_P1.27mm
Connections:
- net labels removed: COM1
