File: hardware/_autosave-ACS DB.kicad_pcb (KiCad board)
At the start: 2 copper layers, 160 x 105 mm, 45 parts, among them IC1 USR-ES1, J1 Power, J2 Reader 2, J3 Reader 1, J4 Relay 1, J5 Sensor 1, J6 Relay 2, J7 Sensor 2, J8 PB2, J9 PB1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

Commit message: update pcb layout
Parts:
- moved H4 190.3 mm to (230.0, 50.0)
- moved H3 165.8 mm to (230.0, 145.0)
- moved H1 89.0 mm to (80.0, 50.0)
- moved H2 23.5 mm to (80.0, 145.0)
- moved IC1 13.9 mm to (100.0, 55.0)
- moved C1 10.0 mm to (171.6, 53.3)
- moved C2 10.0 mm to (134.1, 55.9)
- moved D1 10.0 mm to (160.2, 49.5)
- moved D2 10.0 mm to (192.6, 58.4)
- moved D3 10.0 mm to (199.6, 58.4)
- moved D4 10.0 mm to (185.6, 51.3)
- moved D5 10.0 mm to (199.6, 51.4)
- moved D6 10.0 mm to (192.6, 51.4)
- moved L1 10.0 mm to (145.6, 55.2)
- moved R1 10.0 mm to (190.9, 65.3)
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