File: hardware/ACS DB.kicad_pcb (KiCad board)
At the start: 2 copper layers, 160 x 105 mm, 45 parts, among them IC1 USR-ES1, J1 Power, J2 Reader 2, J3 Reader 1, J4 Relay 1, J5 Sensor 1, J6 Relay 2, J7 Sensor 2, J8 PB2, J9 PB1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

Commit message: add library package
Parts:
- added C3: 22pF, Capacitor_SMD:C_0805_2012Metric_Pad1.18x1.45mm_HandSolder, F.Cu at (177.2, 94.6)
- added C4: 100nF, Capacitor_SMD:C_0805_2012Metric_Pad1.18x1.45mm_HandSolder, F.Cu at (181.0, 98.4)
- added C5: 10uF, Capacitor_SMD:C_0805_2012Metric_Pad1.18x1.45mm_HandSolder, F.Cu at (200.7, 80.6)
- added C6: 100nF, Capacitor_SMD:C_0805_2012Metric_Pad1.18x1.45mm_HandSolder, F.Cu at (198.8, 82.5)
- added F3: MF-MSMF250/X, Resistor_SMD:R_1812_4532Metric_Pad1.30x3.40mm_HandSolder, F.Cu at (146.1, 66.0)
- added U4: ATmega328P-AU, Package_QFP:TQFP-32_7x7mm_P0.8mm, F.Cu at (191.1, 85.7)
- added Y1: Crystal, Crystal:Crystal_SMD_HC49-SD, F.Cu at (182.2, 93.3)
- moved H4 190.3 mm to (230.0, 50.0)
- moved H3 165.8 mm to (230.0, 145.0)
- moved IC1 99.7 mm to (15.2, 68.6)
- moved H1 89.0 mm to (80.0, 50.0)
- moved F1 49.2 mm to (214.6, 121.9), turned to 180 degrees
- moved F2 39.6 mm to (214.6, 77.5)
- moved U3 34.6 mm to (184.2, 108.0)
- moved H2 23.5 mm to (80.0, 145.0)
- moved U2 20.7 mm to (174.6, 64.1)
- moved R4 18.0 mm to (203.2, 66.7)
- moved C2 13.9 mm to (153.7, 66.0), turned to 0 degrees
- moved D5 12.7 mm to (201.9, 61.6)
- moved D6 12.3 mm to (195.6, 61.6)
- moved R2 11.7 mm to (203.2, 55.9)
- moved D3 10.8 mm to (201.9, 50.8)
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Connections:
- D2 pad 1: Net-(D2-Pad1) -> /LED_ACT
- D3 pad 1: Net-(D3-Pad1) -> /LED_IN
- D5 pad 1: /O1 -> /S1
- D6 pad 1: /O2 -> /S2
- J4 pad 1: /NC_1 -> /COM_1
- J4 pad 2: /COM_1 -> /NC_1
- J6 pad 1: /NC_2 -> /COM_2
- J6 pad 2: /COM_2 -> /NC_2
- R4 pad 1: +12V -> +5V
- R5 pad 1: +12V -> +5V
- U2 pad 3: GND -> Net-(U2-Pad3)
Routing:
- net +12V: track 0.00 -> 337.5 mm
- net /NC_2: track 0.00 -> 24.1 mm
- net /NC_1: track 0.00 -> 23.2 mm
- net +5V: track 0.00 -> 22.9 mm
- net /COM_1: track 0.00 -> 19.3 mm
- net /COM_2: track 0.00 -> 18.5 mm
- net /D0_1: track 0.00 -> 17.7 mm
- net /LED_1: track 0.00 -> 17.7 mm
- net /D1_1: track 0.00 -> 17.7 mm
- net /D0_2: track 0.00 -> 17.6 mm
- net /LED_2: track 0.00 -> 17.6 mm
- net /D1_2: track 0.00 -> 17.6 mm
- net /PB1: track 0.00 -> 17.6 mm
- net /XTAL1: track 0.00 -> 17.2 mm
- net /S2: track 0.00 -> 16.7 mm
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- added copper zone on B.Cu, net GND
- added copper zone on F.Cu, net GND
Other:
- net class Power 5V added: clearance 0.2, trace_width 1.36652, via_dia 0.8, via_drill 0.4
- net class Signal added: clearance 0.2, trace_width 0.25, via_dia 0.8, via_drill 0.4
- net class power 12V added: clearance 0.2, trace_width 0.795068, via_dia 0.8, via_drill 0.4
- board text added: "+12V"
- board text added: "COM"
- board text added: "D0"
- board text added: "D1"
- board text added: "GND"
- board text added: "LED"
- board text added: "NC"
- board text added: "NO"
- board text added: "PB1"
- board text added: "PB2"
- board text added: "S1"
- board text added: "S2"
