File: hardware/_autosave-ACS DB.sch (KiCad schematic (older format))
At the start: 52 parts, among them IC1 USR-ES1, J1 Power, J2 Reader 2, J3 Reader 1, J4 Relay 1, J5 Sensor 1, J6 Relay 2, J7 Sensor 2, J8 PB2, J9 PB1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

Commit message: add library package
Changed lines of the file:
@@
 	9325 3875 9600 3875
-Wire Wire Line
-	9325 3975 9600 3975
 Wire Wire Line
 	9325 4075 9600 4075
@@
 GND
 Text Label 9350 3875 0    50   ~ 0
-NC_1
-Text Label 9350 3975 0    50   ~ 0
 COM_1
 Text Label 9350 4075 0    50   ~ 0
 NO_1
 Wire Wire Line
+	9325 5325 9600 5325
+Wire Wire Line
 	9325 5225 9600 5225
 Wire Wire Line
-	9325 5325 9600 5325
-Wire Wire Line
 	9325 5425 9600 5425
+Text Label 9350 5325 0    50   ~ 0
+NC_2
 Text Label 9350 5225 0    50   ~ 0
-NC_2
-Text Label 9350 5325 0    50   ~ 0
 COM_2
 Text Label 9350 5425 0    50   ~ 0
@@
 Text Label 6150 2500 0    50   ~ 0
 LED_IN
+Wire Wire Line
+	9325 3975 9600 3975
+Text Label 9350 3975 0    50   ~ 0
+NC_1
 $EndSCHEMATC
